File: dancing_forest.kicad_pcb (KiCad board)
At the start: 4 copper layers, 148 x 148 mm, 177 parts, among them J1 USB_C_Receptacle_USB2.0, J10 Conn_01x05, J11 Conn_01x05, J12 Conn_01x05, J13 Conn_01x05, J14 Conn_01x05, J15 Conn_01x02, J16 Conn_01x04, J2 Conn_01x01, J3 Conn_01x01, J4 SM04B-SRSS-TB(LF)(SN), J5 Conn_01x03, J6 Conn_01x04, J7 Conn_01x01, J8 Conn_01x01, J9 Conn_01x05, Q1 AO3400A, Q2 AO3400A, U1 TXS0101DCKR, U11 TXS0101DCKR, U12 INA199xxDCK, U13 ESP32-S3-MINI-1-N8, U2 TXS0101DCKR, U3 LD1086DT33TR, U4 FT231XS, U5 LSM6DS3, U6 TXS0101DCKR, U7 DW01, U8 TP4056, U9 FS8205A

Commit message: Updated files including PCB fix. Added license.
Parts:
- removed C11: 0.1uF, Capacitor_SMD:C_0805_2012Metric
- removed J13, J14: Conn_01x05, Connector_PinHeader_1.27mm:PinHeader_1x05_P1.27mm_Vertical
- removed REF** (x3): breakaway, led:breakaway
- added C25: 0.1uF, Capacitor_SMD:C_0603_1608Metric, B.Cu at (136.5, 163.2)
- added C26: 0.1uF, Capacitor_SMD:C_0603_1608Metric, B.Cu at (104.6, 247.3)
- added C27: 1u, Capacitor_SMD:C_0603_1608Metric, B.Cu at (104.6, 249.8)
- added G***: LOGO, led:artwork_smaller, B.Cu at (289.1, 191.5)
- added H10: MountingHole_3.2mm_Plastite_#4, H10, F.Cu at (250.6, 229.1)
- added H11: MountingHole_3.2mm_Plastite_#4, H11, F.Cu at (250.6, 170.9)
- added H12: MountingHole_3.2mm_Plastite_#4, H12, F.Cu at (329.4, 170.9)
- added H4: MountingHole, led:MountingHole_3.2mm_Plastite_#4, F.Cu at (175.7, 170.9)
- added H5: MountingHole, led:MountingHole_3.2mm_Plastite_#4, F.Cu at (320.8, 217.5)
- added H6: MountingHole, led:MountingHole_3.2mm_Plastite_#4, F.Cu at (259.2, 217.5)
- added H7: MountingHole, led:MountingHole_3.2mm_Plastite_#4, F.Cu at (259.2, 182.5)
- added H8: MountingHole, led:MountingHole_3.2mm_Plastite_#4, F.Cu at (320.8, 182.5)
- added H9: MountingHole_3.2mm_Plastite_#4, H9, F.Cu at (329.4, 229.1)
- added J19: Conn_01x01, led:spring_F6-6-4-0.4Z, F.Cu at (273.0, 203.5)
- added J20: Conn_01x01, led:spring_F6-6-4-0.4Z, F.Cu at (307.0, 203.5)
- added JP8: SolderJumper_2_Open, Jumper:SolderJumper-2_P1.3mm_Open_RoundedPad1.0x1.5mm, F.Cu at (121.2, 138.8)
- added JP9: SolderJumper_2_Open, Jumper:SolderJumper-2_P1.3mm_Open_RoundedPad1.0x1.5mm, F.Cu at (121.2, 136.1)
- added Q5: Q_NPN_BEC, Package_TO_SOT_SMD:SOT-23-3, B.Cu at (109.0, 248.7)
- added Q6: Q_NPN_BEC, Package_TO_SOT_SMD:SOT-23-3, B.Cu at (109.0, 244.9)
- added R18: 5.1k, Resistor_SMD:R_0603_1608Metric, B.Cu at (136.7, 156.3)
- added R19: 10k 0.5%, Resistor_SMD:R_0805_2012Metric, B.Cu at (113.3, 244.4)
- added R20: 10k 0.5%, Resistor_SMD:R_0805_2012Metric, B.Cu at (115.0, 239.7)
- added R21: 10k 0.5%, Resistor_SMD:R_0805_2012Metric, B.Cu at (113.5, 249.8)
- added R22: 10k 0.5%, Resistor_SMD:R_0805_2012Metric, B.Cu at (141.0, 152.0)
- added R23: 10k 0.5%, Resistor_SMD:R_0805_2012Metric, B.Cu at (138.8, 152.0)
- added R24: 10k 0.5%, Resistor_SMD:R_0805_2012Metric, B.Cu at (136.6, 152.0)
- added R25: 10k 0.5%, Resistor_SMD:R_0805_2012Metric, B.Cu at (134.4, 152.0)
- added R26: 10k 0.5%, Resistor_SMD:R_0805_2012Metric, B.Cu at (122.5, 143.7)
- added R27: 10k 0.5%, Resistor_SMD:R_0805_2012Metric, B.Cu at (122.5, 141.5)
- added RGBD61: WS2812B, LED_SMD:LED_WS2812B_PLCC4_5.0x5.0mm_P3.2mm, F.Cu at (290.0, 157.0)
- added RGBD62: WS2812B, LED_SMD:LED_WS2812B_PLCC4_5.0x5.0mm_P3.2mm, F.Cu at (311.5, 162.8)
- added RGBD63: WS2812B, LED_SMD:LED_WS2812B_PLCC4_5.0x5.0mm_P3.2mm, F.Cu at (327.2, 178.5)
- added RGBD64: WS2812B, LED_SMD:LED_WS2812B_PLCC4_5.0x5.0mm_P3.2mm, F.Cu at (333.0, 200.0)
- added RGBD65: WS2812B, LED_SMD:LED_WS2812B_PLCC4_5.0x5.0mm_P3.2mm, F.Cu at (327.2, 221.5)
- added RGBD66: WS2812B, LED_SMD:LED_WS2812B_PLCC4_5.0x5.0mm_P3.2mm, F.Cu at (311.5, 237.2)
- added RGBD67: WS2812B, LED_SMD:LED_WS2812B_PLCC4_5.0x5.0mm_P3.2mm, F.Cu at (290.0, 243.0)
- added RGBD68: WS2812B, LED_SMD:LED_WS2812B_PLCC4_5.0x5.0mm_P3.2mm, F.Cu at (268.5, 237.2)
- added RGBD69: WS2812B, LED_SMD:LED_WS2812B_PLCC4_5.0x5.0mm_P3.2mm, F.Cu at (252.8, 221.5)
- added RGBD70: WS2812B, LED_SMD:LED_WS2812B_PLCC4_5.0x5.0mm_P3.2mm, F.Cu at (247.0, 200.0)
- added RGBD71: WS2812B, LED_SMD:LED_WS2812B_PLCC4_5.0x5.0mm_P3.2mm, F.Cu at (252.8, 178.5)
- added RGBD72: WS2812B, LED_SMD:LED_WS2812B_PLCC4_5.0x5.0mm_P3.2mm, F.Cu at (268.5, 162.8)
- added RGBSIDE13: SK6812-SIDE, led:SK6812SIDE, F.Cu at (57.2, 200.0)
- added RGBSIDE14: SK6812-SIDE, led:SK6812SIDE, F.Cu at (59.9, 220.4)
- added RGBSIDE15: SK6812-SIDE, led:SK6812SIDE, F.Cu at (67.8, 239.5)
- added RGBSIDE16: SK6812-SIDE, led:SK6812SIDE, F.Cu at (80.4, 255.9)
- added RGBSIDE17: SK6812-SIDE, led:SK6812SIDE, F.Cu at (96.8, 268.4)
- added RGBSIDE18: SK6812-SIDE, led:SK6812SIDE, F.Cu at (115.8, 276.3)
- added RGBSIDE19: SK6812-SIDE, led:SK6812SIDE, F.Cu at (136.2, 279.0)
- added RGBSIDE20: SK6812-SIDE, led:SK6812SIDE, F.Cu at (156.7, 276.3)
- added RGBSIDE21: SK6812-SIDE, led:SK6812SIDE, F.Cu at (175.8, 268.4)
- added RGBSIDE22: SK6812-SIDE, led:SK6812SIDE, F.Cu at (192.1, 255.9)
- added RGBSIDE23: SK6812-SIDE, led:SK6812SIDE, F.Cu at (204.7, 239.5)
- added RGBSIDE24: SK6812-SIDE, led:SK6812SIDE, F.Cu at (212.6, 220.4)
- added SW1: SW_MEC_5G, led:SW_TS_1101_C_W, F.Cu at (103.2, 234.8)
- added SW2: SW_MEC_5G, led:SW_TS_1101_C_W, F.Cu at (111.4, 241.1)
- added SW3: CONFIG SWITCH, Button_Switch_SMD:SW_DIP_SPSTx06_Slide_KingTek_DSHP06TS_W7.62mm_P1.27mm, F.Cu at (155.0, 134.1)
- added SW4: SW_MEC_5G, led:SW_TS_1101_C_W, F.Cu at (127.7, 136.1)
- added SW5: SW_MEC_5G, led:SW_TS_1101_C_W, F.Cu at (115.9, 136.6)
- added TP1: TestPoint, TestPoint:TestPoint_Keystone_5019_Minature, F.Cu at (154.2, 160.1)
- added TP2: TestPoint, TestPoint:TestPoint_Keystone_5019_Minature, B.Cu at (117.6, 130.6)
- added U10: LIS3MDL, Package_LGA:LGA-12_2x2mm_P0.5mm, B.Cu at (136.9, 159.3)
- added mousebite1: VAL**, mousebite1, F.Cu at (52.0, 200.0)
- added mousebite2: VAL**, mousebite2, F.Cu at (136.2, 115.8)
- added mousebite3: VAL**, mousebite3, F.Cu at (136.2, 284.2)
- added mousebite4: VAL**, mousebite4, F.Cu at (220.5, 200.0)
- added mousebite5: VAL**, mousebite5, F.Cu at (359.5, 200.0)
- added mousebite6: VAL**, mousebite6, F.Cu at (290.0, 130.5)
- added mousebite7: VAL**, mousebite7, F.Cu at (290.0, 269.5)
- C1, C14, C15, C16, C17, C19, C2, C20, C21, C22, C23, C24, C6, D1, D2, J15, J16, J2, J3, J6, J7, J8, RGBD49, RGBD50, RGBD51, RGBD52, RGBD53, RGBD54, RGBD55, RGBD56, RGBD57, RGBD58, RGBD59, RGBD60, U1, U11, U2, U4, U6: moved to F.Cu
- C10: footprint Capacitor_SMD:C_0805_2012Metric -> Capacitor_SMD:C_0603_1608Metric
- C12: value 0.1uF -> 1u; footprint Capacitor_SMD:C_0805_2012Metric -> Capacitor_SMD:C_0603_1608Metric; moved to B.Cu
- C13: footprint Capacitor_SMD:C_0805_2012Metric -> Capacitor_SMD:C_0603_1608Metric; moved to B.Cu
- DIST1, DIST2, DIST3: value VL53L1CXV0FY1 -> Conn_01x05; footprint Sensor_Distance:ST_VL53L1x -> led:5_pin
- H1, H2, H3: footprint led:MountingHole_3.9mm_Plastite_#6 -> led:MountingHole_3.2mm_Plastite_#4
- J10: value Conn_01x05 -> Conn_01x04; footprint Connector_PinHeader_1.27mm:PinHeader_1x05_P1.27mm_Vertical -> Connector_PinHeader_2.00mm:PinHeader_1x04_P2.00mm_Vertical
- J11: value Conn_01x05 -> Upper Connector; footprint Connector_PinHeader_1.27mm:PinHeader_1x05_P1.27mm_Vertical -> Connector_PinSocket_2.00mm:PinSocket_2x06_P2.00mm_Vertical; moved to B.Cu
- J12: value Conn_01x05 -> Lower Connector; footprint Connector_PinHeader_1.27mm:PinHeader_1x05_P1.27mm_Vertical -> Connector_PinHeader_2.00mm:PinHeader_2x06_P2.00mm_Vertical; moved to B.Cu
- J9: value Conn_01x05 -> Conn_01x02; footprint Connector_PinHeader_1.27mm:PinHeader_1x05_P1.27mm_Vertical -> Connector_Molex:Molex_KK-254_AE-6410-02A_1x02_P2.54mm_Vertical; moved to B.Cu
- R16, R17: moved to B.Cu
- U13: footprint Espressif:ESP32-S3-MINI-1 -> esp:ESP32-S3-MINI-1-breakout
- moved RGBD30 210.4 mm to (59.9, 189.9), turned to -97.5 degrees
- moved RGBD31 210.4 mm to (59.9, 210.1), turned to -82.5 degrees
- moved RGBD29 207.3 mm to (65.1, 170.5), turned to -112.5 degrees
- moved RGBD32 207.3 mm to (65.1, 229.5), turned to -67.5 degrees
- moved RGBD28 201.4 mm to (75.2, 153.1), turned to -127.5 degrees
- moved RGBD33 201.4 mm to (75.2, 246.9), turned to -52.5 degrees
- moved RGBD27 192.6 mm to (89.4, 138.9), turned to -142.5 degrees
- moved RGBD34 192.6 mm to (89.4, 261.1), turned to -37.5 degrees
- moved R6 186.1 mm to (76.0, 175.3)
- moved R7 184.4 mm to (76.0, 177.3)
- moved C9 182.8 mm to (76.3, 179.5), turned to 180 degrees
- moved RGBSIDE12 182.8 mm to (59.9, 179.6), turned to -105 degrees
- moved D1 181.9 mm to (75.9, 175.1), turned to 0 degrees
- moved RGBD35 181.2 mm to (106.8, 271.1), turned to -22.5 degrees
- moved RGBD26 181.2 mm to (106.8, 128.9), turned to -157.5 degrees
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Connections:
- net /USB_D+ renamed USB_D+
- net /USB_D- renamed USB_D-
- C13 pad 1: +3V3 -> Net-(U10-C1)
- C8 pad 1: Net-(D1-A) -> VBUS
- D1 pad 2: Net-(D1-A) -> VBUS
- D2 pad 2: Net-(D1-A) -> VBUS
- DIST1 pad 2: GND -> SDA
- DIST1 pad 3: GND -> SCL
- DIST1 pad 4: GND -> XSHUT1
- DIST1 pad 5: XSHUT1 -> GND
- DIST2 pad 2: GND -> SDA
- DIST2 pad 3: GND -> SCL
- DIST2 pad 4: GND -> XSHUT2
- DIST2 pad 5: XSHUT2 -> GND
- DIST3 pad 2: GND -> SDA
- DIST3 pad 3: GND -> SCL
- DIST3 pad 4: GND -> XSHUT3
- DIST3 pad 5: XSHUT3 -> GND
- J10 pad 1: +3V3 -> GND
- J10 pad 2: SDA -> +BATT
- J10 pad 3: SCL -> AUX1
- J10 pad 4: XSHUT1 -> AUX2
- J11 pad 1: +3V3 -> BAT-
- J11 pad 2: SDA -> +BATT
- J11 pad 3: SCL -> BAT-
- J11 pad 4: XSHUT2 -> +BATT
- J11 pad 5: GND -> BAT-
- J12 pad 1: +3V3 -> BAT-
- J12 pad 2: SDA -> +BATT
- J12 pad 3: SCL -> BAT-
- J12 pad 4: XSHUT2 -> +BATT
- J12 pad 5: GND -> BAT-
- J9 pad 1: +3V3 -> +BATT
- J9 pad 2: SDA -> BAT-
- JP1 pad 2: Net-(D1-A) -> VBUS
- RGBD48 pad 2: Net-(RGBD48-DOUT) -> RGB-LOWER-OUT
- RGBD49 pad 4: Net-(RGBD48-DOUT) -> RGB-UPPER-IN
- RGBD55 pad 2: unconnected-(RGBD55-DOUT-Pad2) -> Net-(RGBD55-DOUT)
- RGBD56 pad 4: Net-(RGBD56-DIN) -> Net-(RGBD55-DOUT)
- RGBD60 pad 2: Net-(RGBD1-DIN) -> Net-(RGBD60-DOUT)
- RGBSIDE12 pad 3: Net-(RGBSIDE1-DIN) -> Net-(RGBSIDE12-DOUT)
- RGBSIDE3 pad 3: unconnected-(RGBSIDE3-DOUT-Pad3) -> Net-(RGBSIDE3-DOUT)
- RGBSIDE4 pad 1: Net-(RGBSIDE4-DIN) -> Net-(RGBSIDE3-DOUT)
- RGBWD10 pad 4: unconnected-(RGBWD10-DOUT-Pad4) -> Net-(RGBWD10-DOUT)
- RGBWD11 pad 2: Net-(RGBWD11-DIN) -> Net-(RGBWD10-DOUT)
- RGBWD16 pad 4: Net-(RGBWD1-DIN) -> unconnected-(RGBWD16-DOUT-Pad4)
- U1 pad 4: Net-(RGBD56-DIN) -> Net-(RGBD1-DIN)
- U13 pad 19: unconnected-(U13-GPIO15/U0RTS/ADC2_CH4/XTAL_32K_P-Pad19) -> ADDY_1
- U13 pad 20: unconnected-(U13-GPIO16/U0CTS/ADC2_CH5/XTAL_32K_NH5-Pad20) -> ADDY_2
- U13 pad 21: unconnected-(U13-GPIO17/U1TXD/ADC2_CH6-Pad21) -> ADDY_3
- U13 pad 22: unconnected-(U13-GPIO18/U1RXD/ADC2_CH7/CLK_OUT3-Pad22) -> ADDY_4
- U13 pad 23: unconnected-(U13-GPIO19/U1RTS/ADC2_CH8/CLK_OUT2/USB_D--Pad23) -> DRDY
- U13 pad 24: unconnected-(U13-GPIO20/U1CTS/ADC2_CH9/CLK_OUT1/USB_D+-Pad24) -> INT
- U13 pad 25: unconnected-(U13-GPIO21-Pad25) -> AUX1
- U13 pad 34: unconnected-(U13-GPIO38/FSPIWP/SUBSPIWP-Pad34) -> ADDY_5
- U13 pad 35: unconnected-(U13-MTCK/GPIO39/CLK_OUT3/SUBSPICS1-Pad35) -> ADDY_6
- U13 pad 36: unconnected-(U13-MTDO/GPIO40/CLK_OUT2-Pad36) -> Net-(U13-MTDO/GPIO40/CLK_OUT2)
- U13 pad 37: unconnected-(U13-MTDI/GPIO41/CLK_OUT1-Pad37) -> Net-(U13-MTDI/GPIO41/CLK_OUT1)
- U13 pad 38: unconnected-(U13-MTMS/GPIO42-Pad38) -> AUX2
- U13 pad 4: unconnected-(U13-GPIO0/BOOT-Pad4) -> IO0
- U13 pad 45: +3V3 -> EN
- U2 pad 4: Net-(RGBWD11-DIN) -> Net-(RGBWD1-DIN)
- U4 pad 1: unconnected-(U4-~{DTR}-Pad1) -> ~{DTR}
- U4 pad 2: unconnected-(U4-~{RTS}-Pad2) -> ~{RTS}
- U6 pad 4: Net-(RGBSIDE4-DIN) -> Net-(RGBSIDE1-DIN)
- U8 pad 4: Net-(D1-A) -> VBUS
- U8 pad 8: Net-(D1-A) -> VBUS
- U8 pad 9: Net-(D1-A) -> VBUS
Routing:
- net +BATT: track 1466.6 -> 2243.1 mm, vias 46 -> 65
- net IO0: track 0.00 -> 259.1 mm, vias 0 -> 4
- net EN: track 0.00 -> 192.2 mm, vias 0 -> 1
- net RGB-LOWER-OUT: track 0.00 -> 146.8 mm, vias 0 -> 2
- net XSHUT1: track 231.7 -> 100.6 mm, vias 5 -> 1
- net XSHUT3: track 105.1 -> 229.8 mm, vias 5 -> 1
- net BAT-: track 57.0 -> 166.1 mm, vias 0 -> 2
- net +3V3: track 466.5 -> 568.9 mm
- net RGB-UPPER-IN: track 0.00 -> 87.0 mm, vias 0 -> 1
- net VBUS: track 66.7 -> 152.2 mm, vias 0 -> 2
- net XSHUT2: track 72.8 -> 143.3 mm
- net ESP_TX: track 228.7 -> 167.3 mm, vias 8 -> 1
- net Net-(RGBD48-DOUT): track 57.4 -> 0.00 mm, vias 1 -> 0
- net LEDGND: track 136.6 -> 190.6 mm, vias 94 -> 118
- net ESP_RX: track 211.0 -> 161.9 mm, vias 5 -> 2
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- added copper zone on In1.Cu, net LEDGND
- removed copper zone on F.Cu, net +BATT
- removed copper zone on B.Cu, net Net-(JP4-B)
Other:
- board size 148 x 148 mm -> 322.5 x 183.5 mm
- board text added: "3.3v"
- board text added: "6 5 4 3 2 1"
- board text added: "Address"
- board text added: "Batt"
- board text added: "Charger Disconnect"
- board text added: "Curr meas bypass"
- board text added: "Dancing Forest PCB rev 2, design by Sam Cooler and Taylor Alexander 2023"
- board text added: "Disable Battery Protection"
- board text added: "FLASH"
- board text added: "GND"
- board text added: "RESET"
- board text added: "User Switch 1"
- board text added: "User Switch 2"
- board text added: "aux USB port"
- board text added: "breathe"
- board text added: "burning man here we come!"
- board text added: "energy and grace with a dose of wit the room lights up overalls and angle grinders sparks fly"
- board text added: "feel your body"
- board text added: "from a distance the glow attracts up close there is so much more to discover"
- board text added: "just to see what happens and with it we make beauty and joy"
- board text added: "slow down"
- board text added: "the mind will follow"
- board text added: "this is an adventure"
- board text added: "we did it!"
- board text added: "we're riding this ball we're flying through space round and round we go we have no destination I'm so happy we can enjoy this journey together"
- board text added: "your mind wanders to beautiful places you make them real and invite others"
- board text removed: "+3.3v"
- board text removed: "Batt+"
- board text removed: "Charger connect."
- board text removed: "Current measure bypass."
- board text removed: "Dancing forest PCB rev 1, design by Sam Cooler and Taylor Alexander 2023"
- board text removed: "Disable protection."
- board text removed: "I2C Address"
- board text removed: "Q_PWR"
- board text removed: "You're wonderful!"
