File: dancing_forest.kicad_sch (KiCad schematic)
At the start: 174 parts, among them J1 USB_C_Receptacle_USB2.0, J10 Conn_01x03, J10 Conn_01x05, J11 Conn_01x05, J12 Conn_01x05, J13 Conn_01x05, J14 Conn_01x05, J2 Conn_01x01, J2 Conn_01x04, J3 Conn_01x01, J4 SM04B-SRSS-TB(LF)(SN), J7 Conn_01x01, J7 Conn_01x02, J8 Conn_01x01, J9 Conn_01x05, Q1 AO3400A, Q2 AO3400A, U1 TXS0101DCKR, U11 TXS0101DCKR, U12 INA199xxDCK, U13 ESP32-S3-MINI-1-N8, U2 TXS0101DCKR, U3 LD1086DT33TR, U4 FT231XS, U5 LSM6DS3, U6 TXS0101DCKR, U7 DW01, U8 TP4056, U9 FS8205A

Commit message: Updated files including PCB fix. Added license.
Parts:
- removed C11, C12: 0.1uF, Capacitor_SMD:C_0805_2012Metric, symbol Device:C
- removed DIST1, DIST2, DIST3: VL53L1CXV0FY1, Sensor_Distance:ST_VL53L1x, symbol Sensor_Distance:VL53L1CXV0FY1
- removed H1 (x2): MountingHole, led:MountingHole_3.9mm_Plastite_#6, symbol Mechanical:MountingHole
- removed J10, J11, J13: Conn_01x05, Connector_PinHeader_1.27mm:PinHeader_1x05_P1.27mm_Vertical, symbol Connector_Generic:Conn_01x05
- added C124 (x2): 1u, Capacitor_SMD:C_0603_1608Metric, symbol Device:C
- added C25, C26: 0.1uF, Capacitor_SMD:C_0603_1608Metric, symbol Device:C
- added H1 (x7): MountingHole, led:MountingHole_3.2mm_Plastite_#4, symbol Mechanical:MountingHole
- added J10: Conn_01x04, Connector_PinHeader_2.00mm:PinHeader_1x04_P2.00mm_Vertical, symbol Connector_Generic:Conn_01x04
- added J11: Upper Connector, Connector_PinSocket_2.00mm:PinSocket_2x06_P2.00mm_Vertical, symbol Connector_Generic:Conn_02x06_Odd_Even
- added J12: Lower Connector, Connector_PinHeader_2.00mm:PinHeader_2x06_P2.00mm_Vertical, symbol Connector_Generic:Conn_02x06_Odd_Even
- added J19, J20: Conn_01x01, led:spring_F6-6-4-0.4Z, symbol Connector_Generic:Conn_01x01
- added J7: Conn_01x02, Connector_Molex:Molex_KK-254_AE-6410-02A_1x02_P2.54mm_Vertical, symbol Connector_Generic:Conn_01x02
- added JP8, JP9: SolderJumper_2_Open, Jumper:SolderJumper-2_P1.3mm_Open_RoundedPad1.0x1.5mm, symbol Jumper:SolderJumper_2_Open
- added Q5, Q6: Q_NPN_BEC, Package_TO_SOT_SMD:SOT-23-3, symbol Device:Q_NPN_BEC
- added R18: 5.1k, Resistor_SMD:R_0603_1608Metric, symbol Device:R
- added R19, R20, R21, R22, R23, R24, R25, R26, R27: 10k 0.5%, Resistor_SMD:R_0805_2012Metric, symbol Device:R
- added RGBD61, RGBD62, RGBD63, RGBD64, RGBD65, RGBD66, RGBD67, RGBD68, RGBD69, RGBD70, RGBD71, RGBD72: WS2812B, LED_SMD:LED_WS2812B_PLCC4_5.0x5.0mm_P3.2mm, symbol LED:WS2812B
- added RGBSIDE13, RGBSIDE14, RGBSIDE15, RGBSIDE16, RGBSIDE17, RGBSIDE18, RGBSIDE19, RGBSIDE20, RGBSIDE21, RGBSIDE22, RGBSIDE23, RGBSIDE24: SK6812-SIDE, led:SK6812SIDE, symbol dancing_forest:SK6812-SIDE
- added SW1 (x4): SW_MEC_5G, led:SW_TS_1101_C_W, symbol Switch:SW_Push
- added SW3: CONFIG SWITCH, Button_Switch_SMD:SW_DIP_SPSTx06_Slide_KingTek_DSHP06TS_W7.62mm_P1.27mm, symbol Switch:SW_DIP_x06
- added TP1, TP2: TestPoint, TestPoint:TestPoint_Keystone_5019_Minature, symbol Connector:TestPoint
- added U10: LIS3MDL, Package_LGA:LGA-12_2x2mm_P0.5mm, symbol Sensor_Magnetic:LIS3MDL
- C10, C13: footprint Capacitor_SMD:C_0805_2012Metric -> Capacitor_SMD:C_0603_1608Metric; LCSC C38141 -> C14663
- DIST1: renamed from J9; footprint Connector_PinHeader_1.27mm:PinHeader_1x05_P1.27mm_Vertical -> led:5_pin
- DIST2: renamed from J12; footprint Connector_PinHeader_1.27mm:PinHeader_1x05_P1.27mm_Vertical -> led:5_pin
- DIST3: renamed from J14; footprint Connector_PinHeader_1.27mm:PinHeader_1x05_P1.27mm_Vertical -> led:5_pin
- H1: footprint led:MountingHole_3.9mm_Plastite_#6 -> led:MountingHole_3.2mm_Plastite_#4
- R15: LCSC C236283 -> C104574
- U13: footprint Espressif:ESP32-S3-MINI-1 -> esp:ESP32-S3-MINI-1-breakout
Connections:
- net +3V3: now also C124.1, C25.1, R20.2, R22.1, R23.1, R24.1, R25.1, R26.1, R27.1, U10.10 (~{CS}), U10.5 (Vdd), U10.6 (Vdd_IO); no longer C13.1, U13.45 (EN)
- net +BATT: now also J10.2 (Pin_2), J11.2 (Pin_2), J11.4 (Pin_4), J11.6 (Pin_6), J11.8 (Pin_8), J12.2 (Pin_2), J12.4 (Pin_4), J12.6 (Pin_6), J12.8 (Pin_8), J20.1 (Pin_1), J7.1 (Pin_1), RGBD61.1 (VDD), RGBD62.1 (VDD), RGBD63.1 (VDD), RGBD64.1 (VDD), RGBD65.1 (VDD), RGBD66.1 (VDD), RGBD67.1 (VDD), RGBD68.1 (VDD), RGBD69.1 (VDD), RGBD70.1 (VDD), RGBD71.1 (VDD), RGBD72.1 (VDD), RGBSIDE13.2 (VDD), RGBSIDE14.2 (VDD), RGBSIDE15.2 (VDD), RGBSIDE16.2 (VDD), RGBSIDE17.2 (VDD), RGBSIDE18.2 (VDD), RGBSIDE19.2 (VDD), RGBSIDE20.2 (VDD), RGBSIDE21.2 (VDD), RGBSIDE22.2 (VDD), RGBSIDE23.2 (VDD), RGBSIDE24.2 (VDD)
- net BAT-: now also J11.1 (Pin_1), J11.3 (Pin_3), J11.5 (Pin_5), J11.7 (Pin_7), J12.1 (Pin_1), J12.3 (Pin_3), J12.5 (Pin_5), J12.7 (Pin_7), J19.1 (Pin_1), J7.2 (Pin_2)
- net GND: now also C124.2, C124.2, C25.2, C26.2, J10.1 (Pin_1), JP8.1 (A), JP9.1 (A), R18.1, SW1.1, SW1.1, SW1.1, SW1.1, SW3.1, SW3.2, SW3.3, SW3.4, SW3.5, SW3.6, TP1.1, TP2.1, U10.12 (GND), U10.2 (GND), U10.3 (GND)
- net LEDGND: now also J11.11 (Pin_11), J11.9 (Pin_9), J12.11 (Pin_11), J12.9 (Pin_9), RGBD61.3 (VSS), RGBD62.3 (VSS), RGBD63.3 (VSS), RGBD64.3 (VSS), RGBD65.3 (VSS), RGBD66.3 (VSS), RGBD67.3 (VSS), RGBD68.3 (VSS), RGBD69.3 (VSS), RGBD70.3 (VSS), RGBD71.3 (VSS), RGBD72.3 (VSS), RGBSIDE13.4 (VSS), RGBSIDE14.4 (VSS), RGBSIDE15.4 (VSS), RGBSIDE16.4 (VSS), RGBSIDE17.4 (VSS), RGBSIDE18.4 (VSS), RGBSIDE19.4 (VSS), RGBSIDE20.4 (VSS), RGBSIDE21.4 (VSS), RGBSIDE22.4 (VSS), RGBSIDE23.4 (VSS), RGBSIDE24.4 (VSS)
- net SCL: now also U10.1 (SCL/SPC)
- net SDA: now also U10.11 (SDA/SDI/SDO)
- net VBUS: now also C8.1, D1.2 (A), D2.2 (A), JP1.2 (B), U8.4 (VCC), U8.8 (CE), U8.9 (PP)
- net at U2.4 (B): now also RGBWD1.2 (DIN); no longer RGBWD11.2 (DIN)
- net RGB-LOWER-OUT: now reaches RGBD48.2 (DOUT)
- net RGB-LOWER-OUT: now also J12.10 (Pin_10), J12.12 (Pin_12); no longer RGBD49.4 (DIN)
- net at RGBD1.4 (DIN): now also U1.4 (B); no longer RGBD60.2 (DOUT)
- net at RGBWD10.4 (DOUT): now also RGBWD11.2 (DIN)
- net at RGBD56.4 (DIN): now also RGBD55.2 (DOUT); no longer U1.4 (B)
- net at RGBSIDE3.3 (DOUT): now also RGBSIDE4.1 (DIN)
- net at RGBSIDE12.3 (DOUT): now also RGBSIDE13.1 (DIN); no longer RGBSIDE1.1 (DIN)
- net ~{DTR}: now reaches U4.1 (~{DTR})
- net ~{DTR}: now also Q6.2 (E), R21.1
- net ~{RTS}: now reaches U4.2 (~{RTS})
- net ~{RTS}: now also Q5.2 (E), R19.2
- net at U6.4 (B): now also RGBSIDE1.1 (DIN); no longer RGBSIDE4.1 (DIN)
- net at RGBWD16.4 (DOUT): no longer RGBWD1.2 (DIN)
- net ADDY_1: now reaches U13.19 (GPIO15/U0RTS/ADC2_CH4/XTAL_32K_P)
- net ADDY_1: now also R22.2, SW3.12
- net ADDY_2: now reaches U13.20 (GPIO16/U0CTS/ADC2_CH5/XTAL_32K_NH5)
- net ADDY_2: now also R23.2, SW3.11
- net ADDY_3: now reaches U13.21 (GPIO17/U1TXD/ADC2_CH6)
- net ADDY_3: now also R24.2, SW3.10
- net ADDY_4: now reaches U13.22 (GPIO18/U1RXD/ADC2_CH7/CLK_OUT3)
- net ADDY_4: now also R25.2, SW3.9
- net DRDY: now reaches U13.23 (GPIO19/U1RTS/ADC2_CH8/CLK_OUT2/USB_D-)
- net DRDY: now also U10.8 (DRDY)
- net INT: now reaches U13.24 (GPIO20/U1CTS/ADC2_CH9/CLK_OUT1/USB_D+)
- net INT: now also U10.7 (INT)
- net AUX1: now reaches U13.25 (GPIO21)
- net AUX1: now also J10.3 (Pin_3), JP9.2 (B)
- net ADDY_5: now reaches U13.34 (GPIO38/FSPIWP/SUBSPIWP)
- net ADDY_5: now also R26.2, SW3.8
- net ADDY_6: now reaches U13.35 (MTCK/GPIO39/CLK_OUT3/SUBSPICS1)
- net ADDY_6: now also R27.2, SW3.7
- net at U13.36 (MTDO/GPIO40/CLK_OUT2): now also SW1.2
- net at U13.37 (MTDI/GPIO41/CLK_OUT1): now also SW1.2
- net AUX2: now reaches U13.38 (MTMS/GPIO42)
- net AUX2: now also J10.4 (Pin_4), JP8.2 (B)
- net IO0: now reaches U13.4 (GPIO0/BOOT)
- net IO0: now also Q6.3 (C), SW1.2
- new net: RGBD66.2 (DOUT), RGBD67.4 (DIN)
- new net: RGBD65.2 (DOUT), RGBD66.4 (DIN)
- new net: RGBD62.2 (DOUT), RGBD63.4 (DIN)
- new net: RGBD61.2 (DOUT), RGBD62.4 (DIN)
- new net: Q5.1 (B), R21.2
- new net: RGBSIDE14.3 (DOUT), RGBSIDE15.1 (DIN)
- new net: RGBSIDE15.3 (DOUT), RGBSIDE16.1 (DIN)
- new net: RGBSIDE22.3 (DOUT), RGBSIDE23.1 (DIN)
- new net: RGBSIDE23.3 (DOUT), RGBSIDE24.1 (DIN)
- new net: RGBSIDE18.3 (DOUT), RGBSIDE19.1 (DIN)
- new net: RGBSIDE19.3 (DOUT), RGBSIDE20.1 (DIN)
- new net: RGBD67.2 (DOUT), RGBD68.4 (DIN)
- new net: Q6.1 (B), R19.1
- new net: RGBD69.2 (DOUT), RGBD70.4 (DIN)
- new net: RGBD68.2 (DOUT), RGBD69.4 (DIN)
- new net: RGBSIDE20.3 (DOUT), RGBSIDE21.1 (DIN)
- new net: C13.1, U10.4 (C1)
- new net: R18.2, U10.9 (SDO/SA1)
- new net: RGBSIDE13.3 (DOUT), RGBSIDE14.1 (DIN)
- new net: RGBD64.2 (DOUT), RGBD65.4 (DIN)
- new net: RGBSIDE21.3 (DOUT), RGBSIDE22.1 (DIN)
- new net: RGBSIDE17.3 (DOUT), RGBSIDE18.1 (DIN)
- new net: RGBD70.2 (DOUT), RGBD71.4 (DIN)
- new net: RGBD71.2 (DOUT), RGBD72.4 (DIN)
- new net: RGBD60.2 (DOUT), RGBD61.4 (DIN)
- new net: RGBD63.2 (DOUT), RGBD64.4 (DIN)
- new net: RGBSIDE16.3 (DOUT), RGBSIDE17.1 (DIN)
- new net EN: C124.1, C26.1, Q5.3 (C), R20.1, SW1.2, U13.45 (EN)
- new net RGB-UPPER-IN: J11.10 (Pin_10), J11.12 (Pin_12), RGBD49.4 (DIN)
Other:
- note added: "AUDIO???"
- note added: "Connect charger jumper (defaulting to on, route trace as cuttable if desired)"
- note added: "GPIO notes from: https://docs.espressif.com/projects/esp-idf/en /latest/esp32s3/api-reference/peripherals/gpio.html Strapping pin: GPIO0, GPIO3, GPIO45 and GPIO46 are strapping pins. For more infomation, please refer to ESP32-S3 datasheet. SPI0/1: GPIO26-32 are usually used for SPI flash and PSRAM and not recommended for other uses. When using Octal Flash or Octal PSRAM or both, GPIO33~37 are con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"
- note added: "General Jumper 1"
- note added: "General Jumper 2"
- note added: "https://dl.espressif.com/dl/schematics/esp32_devkitc_v4-sch-20180607a.pdf"
- note added: "https://docs.espressif.com/projects/esptool/en/latest/esp32s3/advanced-topics/boot-mode-selection.html"
- note removed: "Connect charger."
- note removed: "TODO: FINALIZE INT1/INT2 pins"
- note removed: "TODO: MAKE SURE BOARD CAN RUN OFF USB WITH NO BATTERY"
- note removed: "TODO: confirm USB footprint before ordering"
- moved on the sheet: C14, C24, C3, C4, C5, C6, J1, J2, JP3, JP6, JP7, R10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
